Commit message: */*

File: install/lg-robot/share/lg-robot/urdf/lgrobot.urdf.xacro (robot description, xacro)
@@ -233,15 +233,85 @@
     </joint>
     //============Plugins==========//
+    <!-- <plugin name="gazebo_ros2_control" filename="libgazebo_ros2_control.so">
+        <robot_param>robot_description</robot_param>
+        <robot_param_node>robot_state_publisher</robot_param_node>
+        <parameters>$(find lg-robot)/config/lg_robot_controllers.yaml</parameters>
+    </plugin> -->
+    <ros2_control name="GazeboSystem" type="system">
+        <hardware>
+            <plugin>
+                gazebo_ros2_control/GazeboSystem
+            </plugin>
+        </hardware>
+        <joint name="joint_leg00">
+            <command_interface name="position"/>
+            <state_interface name="position">
+                <param name="initial_value">0.0</param>
+            </state_interface>
+            <state_interface name="velocity"/>
+        </joint>
+        <joint name="joint_leg00b">
+            <command_interface name="position"/>
+            <state_interface name="position">
+                <param name="initial_value">0.0</param>
+            </state_interface>
+            <state_interface name="velocity"/>
+        </joint>
+        <joint name="joint_leg01">
+            <command_interface name="position"/>
+            <state_interface name="position">
+                <param name="initial_value">0.0</param>
+            </state_interface>
+            <state_interface name="velocity"/>
+        </joint>
+        <joint name="joint_leg01b">
+            <command_interface name="position"/>
+            <state_interface name="position">
+                <param name="initial_value">0.0</param>
+            </state_interface>
+            <state_interface name="velocity"/>
+        </joint>
+        <joint name="joint_leg10">
+            <param name="mimic">joint_leg01</param>
+            <param name="multiplier">1</param>
+            <command_interface name="position"/>
+            <state_interface name="position">
+                <param name="initial_value">0.0</param>
+            </state_interface>
+            <state_interface name="velocity"/>
+        </joint>
+        <joint name="joint_leg10b">
+            <param name="mimic">joint_leg01b</param>
+            <param name="multiplier">1</param>
+            <command_interface name="position"/>
+            <state_interface name="position">
+                <param name="initial_value">0.0</param>
+            </state_interface>
+            <state_interface name="velocity"/>
+        </joint>
+        <joint name="joint_leg11">
+            <param name="mimic">joint_leg00</param>
+            <param name="multiplier">1</param>
+            <command_interface name="position"/>
+            <state_interface name="position">
+                <param name="initial_value">0.0</param>
+            </state_interface>
+            <state_interface name="velocity"/>
+        </joint>
+        <joint name="joint_leg11b">
+            <param name="mimic">joint_leg00b</param>
+            <param name="multiplier">1</param>
+            <command_interface name="position"/>
+            <state_interface name="position">
+                <param name="initial_value">0.0</param>
+            </state_interface>
+            <state_interface name="velocity"/>
+        </joint>
+    </ros2_control>
     <gazebo>
-        <plugin name="gazebo_ros_control" filename="libgazebo_ros_control.so"/>
+        <plugin name="gazebo_ros2_control" filename="libgazebo_ros2_control.so">
+            <parameters>$(find lg-robot)/config/lg_robot_controllers.yaml</parameters>
+            <robot_namespace>/</robot_namespace>
+        </plugin>
     </gazebo>
-    <transmission name="trans_joint_leg00">
-        <type>transmission_interface/SimpleTransmission</type>
-        <joint name="joint_leg00">
-            <hardwareInterface>EffortJointInterface</hardwareInterface>
-        </joint>
-        <actuator name="actuator_joint_leg00">
-            <mechanicalReduction>1</mechanicalReduction>
-        </actuator>
-    </transmission>
 </robot>
